File: iss_mosh_gaz_sensor.sch (KiCad schematic (older format))
At the start: 9 parts, among them J1 Conn_01x04, P1 Power, P2 Analog, P3 Digital, P4 Digital, P5 CONN_01X01, P6 CONN_01X01, P7 CONN_01X01, P8 CONN_01X01

Commit message: Add LoraWan RN2483 connectic
Parts:
- added J2: Conn_01x08, symbol Connector_Generic:Conn_01x08
- added R1: 2k, symbol Device:R
- added R2: 1k, symbol Device:R
Connections:
- net +3V3: now also J2.3 (Pin_3)
- net GND: now also J2.1 (Pin_1), R1.1
- net 6(**) renamed 6_UART_TX
- net 6_UART_TX: now also R2.1
- net 7 renamed 7_UART_RX
- net 7_UART_RX: now also J2.8 (Pin_8)
- new net: J2.7 (Pin_7), R1.2, R2.2
- no-connect marks 26 -> 24
Other:
- note added: "LoraWan RN2483"
Changed lines of the file:
@@
 5(**)
 Text Label 10550 2400 0    60   ~ 0
-6(**)
+6_UART_TX
 Text Label 10550 2300 0    60   ~ 0
-7
+7_UART_RX
 Text Label 10550 2100 0    60   ~ 0
 8
@@
 NoConn ~ 8900 2700
 NoConn ~ 8900 2800
-NoConn ~ 10550 3000
-NoConn ~ 10550 2900
 NoConn ~ 10550 2800
 NoConn ~ 10550 2700
 NoConn ~ 10550 2600
 NoConn ~ 10550 2500
-NoConn ~ 10550 2400
-NoConn ~ 10550 2300
 NoConn ~ 10550 2100
 NoConn ~ 10550 2000
@@
 Wire Wire Line
 	6900 950  6900 900
+$Comp
+L Connector_Generic:Conn_01x08 J2
+U 1 1 5BD9F3B1
+P 3550 2050
+F 0 "J2" H 3470 1425 50  0000 C CNN
+F 1 "Conn_01x08" H 3470 1516 50  0000 C CNN
+F 2 "" H 3550 2050 50  0001 C CNN
+F 3 "~" H 3550 2050 50  0001 C CNN
+	1    3550 2050
+	-1   0    0    1
+$EndComp
+$Comp
+L power:GND #PWR06
+U 1 1 5BDA0B65
+P 4000 2450
+F 0 "#PWR06" H 4000 2200 50  0001 C CNN
+F 1 "GND" H 4000 2300 50  0000 C CNN
+F 2 "" H 4000 2450 50  0000 C CNN
+F 3 "" H 4000 2450 50  0000 C CNN
+	1    4000 2450
+	1    0    0    -1
+$EndComp
+Wire Wire Line
+	3750 2350 4000 2350
+Wire Wire Line
+	4000 2350 4000 2450
+$Comp
+L power:+3.3V #PWR05
+U 1 1 5BDA1FA5
+P 4000 2150
+F 0 "#PWR05" H 4000 2000 50  0001 C CNN
+F 1 "+3.3V" V 3950 2200 50  0000 C CNN
+F 2 "" H 4000 2150 50  0000 C CNN
+F 3 "" H 4000 2150 50  0000 C CNN
+	1    4000 2150
+	0    1    1    0
+$EndComp
+Wire Wire Line
+	3750 2150 4000 2150
+Wire Wire Line
+	3750 1650 4000 1650
+Text Label 4800 1750 0    60   ~ 0
+6_UART_TX
+Text Label 4000 1650 0    60   ~ 0
+7_UART_RX
+Wire Wire Line
+	4800 1750 4700 1750
+$Comp
+L Device:R R2
+U 1 1 5BDA8A22
+P 4550 1750
+F 0 "R2" V 4343 1750 50  0000 C CNN
+F 1 "1k" V 4434 1750 50  0000 C CNN
+F 2 "" V 4480 1750 50  0001 C CNN
+F 3 "~" H 4550 1750 50  0001 C CNN
+	1    4550 1750
+	0    1    1    0
+$EndComp
+$Comp
+L Device:R R1
+U 1 1 5BDA8AA1
+P 4300 1950
+F 0 "R1" H 4230 1904 50  0000 R CNN
+F 1 "2k" H 4230 1995 50  0000 R CNN
+F 2 "" V 4230 1950 50  0001 C CNN
+F 3 "~" H 4300 1950 50  0001 C CNN
+	1    4300 1950
+	-1   0    0    1
+$EndComp
+$Comp
+L power:GND #PWR07
+U 1 1 5BDA8B1A
+P 4300 2150
+F 0 "#PWR07" H 4300 1900 50  0001 C CNN
+F 1 "GND" H 4300 2000 50  0000 C CNN
+F 2 "" H 4300 2150 50  0000 C CNN
+F 3 "" H 4300 2150 50  0000 C CNN
+	1    4300 2150
+	1    0    0    -1
+$EndComp
+Wire Wire Line
+	4300 2150 4300 2100
+Wire Wire Line
+	3750 1750 4300 1750
+Wire Wire Line
+	4300 1800 4300 1750
+Wire Wire Line
+	4300 1750 4400 1750
+NoConn ~ 10550 2900
+NoConn ~ 10550 3000
+Wire Notes Line
+	3350 700  5300 700
+Wire Notes Line
+	5300 700  5300 3600
+Wire Notes Line
+	3350 3600 3350 700
+Wire Notes Line
+	3350 3600 5300 3600
+Connection ~ 4300 1750
+Text Notes 3750 900  0    94   ~ 0
+LoraWan RN2483
 $EndSCHEMATC

Commit message: gas_sensor_schema
not all done, half way to success :)
Parts:
- added C1, C2, C3: 100n, symbol Device:C
- added C4: 1u, symbol Device:C
- added R1, R3: 100k, symbol Device:R
- added R5: 10k, symbol Device:R
- added R6: 1k, symbol Device:R
- added R?: Rcal1, symbol Device:R
- added R?: Rcal2, symbol Device:R
- added U?: LTC1050, symbol Gaz-sensor:LTC1050
Connections:
- net +5V: now also C3.1, U?.7 (V+)
- net A0: now also R5.2
- net GND: now also C1.1, C2.2, C3.2, R1.2, R?.2, U?.4 (V-)
- net 13(SCK) renamed arduino
- net arduino: now also C2.1, R6.1
- new net: C1.2, R1.1, R5.1, U?.3 (+IN)
- new net: C4.1, R3.1, R?.1, U?.2 (-IN)
- new net: R?.1, R?.2
- new net: C4.2, R3.2, R6.2, U?.6 (OUT)
Other:
- moved on the sheet: J1, J2, R1, R2

Commit message: gaz sensor(not done)
Parts:
- gave numbers to parts that had none: 3
Other:
- moved on the sheet: J2, R1, R2
Changed lines of the file:
@@
 L Connector_Generic:Conn_01x08 J2
 U 1 1 5BD9F3B1
-P 9000 4850
-F 0 "J2" H 8920 4225 50  0000 C CNN
-F 1 "Conn_01x08" H 8920 4316 50  0000 C CNN
-F 2 "" H 9000 4850 50  0001 C CNN
-F 3 "~" H 9000 4850 50  0001 C CNN
-	1    9000 4850
+P 900 4750
+F 0 "J2" H 820 4125 50  0000 C CNN
+F 1 "Conn_01x08" H 820 4216 50  0000 C CNN
+F 2 "" H 900 4750 50  0001 C CNN
+F 3 "~" H 900 4750 50  0001 C CNN
+	1    900  4750
 	-1   0    0    1
 $EndComp
@@
 L power:GND #PWR06
 U 1 1 5BDA0B65
-P 9450 5250
-F 0 "#PWR06" H 9450 5000 50  0001 C CNN
-F 1 "GND" H 9450 5100 50  0000 C CNN
-F 2 "" H 9450 5250 50  0000 C CNN
-F 3 "" H 9450 5250 50  0000 C CNN
-	1    9450 5250
-	1    0    0    -1
-$EndComp
-Wire Wire Line
-	9200 5150 9450 5150
-Wire Wire Line
-	9450 5150 9450 5250
+P 1350 5150
+F 0 "#PWR06" H 1350 4900 50  0001 C CNN
+F 1 "GND" H 1350 5000 50  0000 C CNN
+F 2 "" H 1350 5150 50  0000 C CNN
+F 3 "" H 1350 5150 50  0000 C CNN
+	1    1350 5150
+	1    0    0    -1
+$EndComp
+Wire Wire Line
+	1100 5050 1350 5050
+Wire Wire Line
+	1350 5050 1350 5150
 $Comp
 L power:+3.3V #PWR05
 U 1 1 5BDA1FA5
-P 9450 4950
-F 0 "#PWR05" H 9450 4800 50  0001 C CNN
-F 1 "+3.3V" V 9400 5000 50  0000 C CNN
-F 2 "" H 9450 4950 50  0000 C CNN
-F 3 "" H 9450 4950 50  0000 C CNN
-	1    9450 4950
-	0    1    1    0
-$EndComp
-Wire Wire Line
-	9200 4950 9450 4950
-Wire Wire Line
-	9200 4450 9450 4450
-Text Label 10250 4550 0    60   ~ 0
+P 1350 4850
+F 0 "#PWR05" H 1350 4700 50  0001 C CNN
+F 1 "+3.3V" V 1300 4900 50  0000 C CNN
+F 2 "" H 1350 4850 50  0000 C CNN
+F 3 "" H 1350 4850 50  0000 C CNN
+	1    1350 4850
+	0    1    1    0
+$EndComp
+Wire Wire Line
+	1100 4850 1350 4850
+Wire Wire Line
+	1100 4350 1350 4350
+Text Label 2150 4450 0    60   ~ 0
 6_UART_TX
-Text Label 9450 4450 0    60   ~ 0
+Text Label 1350 4350 0    60   ~ 0
 7_UART_RX
 Wire Wire Line
-	10250 4550 10150 4550
+	2150 4450 2050 4450
 $Comp
 L Device:R R2
 U 1 1 5BDA8A22
-P 10000 4550
-F 0 "R2" V 9793 4550 50  0000 C CNN
-F 1 "1k" V 9884 4550 50  0000 C CNN
-F 2 "" V 9930 4550 50  0001 C CNN
-F 3 "~" H 10000 4550 50  0001 C CNN
-	1    10000 4550
+P 1900 4450
+F 0 "R2" V 1693 4450 50  0000 C CNN
+F 1 "1k" V 1784 4450 50  0000 C CNN
+F 2 "" V 1830 4450 50  0001 C CNN
+F 3 "~" H 1900 4450 50  0001 C CNN
+	1    1900 4450
 	0    1    1    0
 $EndComp
@@
 L Device:R R1
 U 1 1 5BDA8AA1
-P 9750 4750
-F 0 "R1" H 9680 4704 50  0000 R CNN
-F 1 "2k" H 9680 4795 50  0000 R CNN
-F 2 "" V 9680 4750 50  0001 C CNN
-F 3 "~" H 9750 4750 50  0001 C CNN
-	1    9750 4750
+P 1650 4650
+F 0 "R1" H 1580 4604 50  0000 R CNN
+F 1 "2k" H 1580 4695 50  0000 R CNN
+F 2 "" V 1580 4650 50  0001 C CNN
+F 3 "~" H 1650 4650 50  0001 C CNN
+	1    1650 4650
 	-1   0    0    1
 $EndComp
@@
 L power:GND #PWR07
 U 1 1 5BDA8B1A
-P 9750 4950
-F 0 "#PWR07" H 9750 4700 50  0001 C CNN
-F 1 "GND" H 9750 4800 50  0000 C CNN
-F 2 "" H 9750 4950 50  0000 C CNN
-F 3 "" H 9750 4950 50  0000 C CNN
-	1    9750 4950
-	1    0    0    -1
-$EndComp
-Wire Wire Line
-	9750 4950 9750 4900
-Wire Wire Line
-	9200 4550 9750 4550
-Wire Wire Line
-	9750 4600 9750 4550
-Wire Wire Line
-	9750 4550 9850 4550
+P 1650 4850
+F 0 "#PWR07" H 1650 4600 50  0001 C CNN
+F 1 "GND" H 1650 4700 50  0000 C CNN
+F 2 "" H 1650 4850 50  0000 C CNN
+F 3 "" H 1650 4850 50  0000 C CNN
+	1    1650 4850
+	1    0    0    -1
+$EndComp
+Wire Wire Line
+	1650 4850 1650 4800
+Wire Wire Line
+	1100 4450 1650 4450
+Wire Wire Line
+	1650 4500 1650 4450
+Wire Wire Line
+	1650 4450 1750 4450
 NoConn ~ 10550 2900
 NoConn ~ 10550 3000
 Wire Notes Line
-	8800 3500 10750 3500
+	700  3400 2650 3400
 Wire Notes Line
-	10750 3500 10750 6400
+	2650 3400 2650 6300
 Wire Notes Line
-	8800 6400 8800 3500
+	700  6300 700  3400
 Wire Notes Line
-	8800 6400 10750 6400
-Connection ~ 9750 4550
-Text Notes 9200 3700 0    94   ~ 0
+	700  6300 2650 6300
+Connection ~ 1650 4450
+Text Notes 1100 3600 0    94   ~ 0
 LoraWan RN2483
 $Comp
@@
 $EndComp
 $Comp
-L Device:R R?
+L Device:R Rcal1
 U 1 1 5BF809A8
 P 2550 1950
-F 0 "R?" V 2343 1950 50  0000 C CNN
+F 0 "Rcal1" V 2343 1950 50  0000 C CNN
 F 1 "Rcal1" V 2434 1950 50  0000 C CNN
 F 2 "" V 2480 1950 50  0001 C CNN
@@
 $EndComp
 $Comp
-L Device:R R?
+L Device:R Rcal2
 U 1 1 5BF881B3
 P 2200 1950
-F 0 "R?" V 1993 1950 50  0000 C CNN
+F 0 "Rcal2" V 1993 1950 50  0000 C CNN
 F 1 "Rcal2" V 2084 1950 50  0000 C CNN
 F 2 "" V 2130 1950 50  0001 C CNN
@@
 $EndComp
 $Comp
-L Gaz-sensor:LTC1050 U?
+L Gaz-sensor:LTC1050 U1
 U 1 1 5BF8822B
 P 3200 2350
-F 0 "U?" H 3450 2250 50  0000 L CNN
+F 0 "U1" H 3450 2250 50  0000 L CNN
 F 1 "LTC1050" H 3300 2150 50  0000 L CNN
 F 2 "" H 2750 2750 50  0001 C CNN
@@
 $EndComp
 $Comp
-L power:GND #PWR?
+L power:GND #PWR0106
 U 1 1 5BF9A2C9
 P 2600 2750
-F 0 "#PWR?" H 2600 2500 50  0001 C CNN
+F 0 "#PWR0106" H 2600 2500 50  0001 C CNN
 F 1 "GND" H 2600 2600 50  0000 C CNN
 F 2 "" H 2600 2750 50  0000 C CNN
@@
 $EndComp
 $Comp
-L power:GND #PWR?
+L power:GND #PWR0107
 U 1 1 5BF9A2FA
 P 2250 2750
-F 0 "#PWR?" H 2250 2500 50  0001 C CNN
+F 0 "#PWR0107" H 2250 2500 50  0001 C CNN
 F 1 "GND" H 2250 2600 50  0000 C CNN
 F 2 "" H 2250 2750 50  0000 C CNN
@@
 $EndComp
 $Comp
-L power:GND #PWR?
+L power:GND #PWR0108
 U 1 1 5BF9A377
 P 3150 2600
-F 0 "#PWR?" H 3150 2350 50  0001 C CNN
+F 0 "#PWR0108" H 3150 2350 50  0001 C CNN
 F 1 "GND" H 3150 2450 50  0000 C CNN
 F 2 "" H 3150 2600 50  0000 C CNN
@@
 $EndComp
 $Comp
-L power:+5V #PWR?
+L power:+5V #PWR0109
 U 1 1 5BF9A3F4
 P 3150 1450
-F 0 "#PWR?" H 3150 1300 50  0001 C CNN
+F 0 "#PWR0109" H 3150 1300 50  0001 C CNN
 F 1 "+5V" V 3150 1650 50  0000 C CNN
 F 2 "" H 3150 1450 50  0000 C CNN
@@
 $EndComp
 $Comp
-L power:GND #PWR?
+L power:GND #PWR0110
 U 1 1 5BF9A506
 P 3350 1800
-F 0 "#PWR?" H 3350 1550 50  0001 C CNN
+F 0 "#PWR0110" H 3350 1550 50  0001 C CNN
 F 1 "GND" H 3350 1650 50  0000 C CNN
 F 2 "" H 3350 1800 50  0000 C CNN
@@
 	1950 2750 1950 3000
 $Comp
-L power:GND #PWR?
+L power:GND #PWR0111
 U 1 1 5BFBB6B6
 P 2050 1950
-F 0 "#PWR?" H 2050 1700 50  0001 C CNN
+F 0 "#PWR0111" H 2050 1700 50  0001 C CNN
 F 1 "GND" H 2050 1800 50  0000 C CNN
 F 2 "" H 2050 1950 50  0000 C CNN
@@
 	5000 2050 5250 2050
 $Comp
-L power:GND #PWR?
+L power:GND #PWR0112
 U 1 1 5BF7680B
 P 5000 2500
-F 0 "#PWR?" H 5000 2250 50  0001 C CNN
+F 0 "#PWR0112" H 5000 2250 50  0001 C CNN
 F 1 "GND" H 5000 2350 50  0000 C CNN
 F 2 "" H 5000 2500 50  0000 C CNN

Commit message: name change for R1
Parts:
- renumbered R1 to R01, R2 to R02
Changed lines of the file:
@@
 	2150 4450 2050 4450
 $Comp
-L Device:R R2
+L Device:R R02
 U 1 1 5BDA8A22
 P 1900 4450
-F 0 "R2" V 1693 4450 50  0000 C CNN
+F 0 "R02" V 1693 4450 50  0000 C CNN
 F 1 "1k" V 1784 4450 50  0000 C CNN
 F 2 "" V 1830 4450 50  0001 C CNN
@@
 $EndComp
 $Comp
-L Device:R R1
+L Device:R R01
 U 1 1 5BDA8AA1
 P 1650 4650
-F 0 "R1" H 1580 4604 50  0000 R CNN
+F 0 "R01" H 1580 4604 50  0000 R CNN
 F 1 "2k" H 1580 4695 50  0000 R CNN
 F 2 "" V 1580 4650 50  0001 C CNN

Commit message: Add footprint of components
Parts:
- C1, C2, C3, C4: footprint (none) -> Capacitor_THT:CP_Axial_L10.0mm_D4.5mm_P15.00mm_Horizontal
- J1: footprint (none) -> Connector_PinSocket_2.54mm:PinSocket_1x04_P2.54mm_Vertical
- J2: footprint (none) -> Connector_PinSocket_2.54mm:PinSocket_1x08_P2.54mm_Vertical
- R01, R02, R1, R3, R5, R6, Rcal1, Rcal2: footprint (none) -> Resistor_THT:R_Axial_DIN0204_L3.6mm_D1.6mm_P5.08mm_Horizontal
- U1: footprint (none) -> Package_DIP:DIP-8_W7.62mm_LongPads; symbol Gaz-sensor:LTC1050 -> iss_mosh_gaz_sensor-rescue:LTC1050-Gaz-sensor
Changed lines of the file:
@@
 F 0 "J1" H 920 1717 50  0000 C CNN
 F 1 "Conn_01x04" H 920 1626 50  0000 C CNN
-F 2 "" H 1000 1400 50  0001 C CNN
+F 2 "Connector_PinSocket_2.54mm:PinSocket_1x04_P2.54mm_Vertical" H 1000 1400 50  0001 C CNN
 F 3 "~" H 1000 1400 50  0001 C CNN
 	1    1000 1400
@@
 F 0 "J2" H 820 4125 50  0000 C CNN
 F 1 "Conn_01x08" H 820 4216 50  0000 C CNN
-F 2 "" H 900 4750 50  0001 C CNN
+F 2 "Connector_PinSocket_2.54mm:PinSocket_1x08_P2.54mm_Vertical" H 900 4750 50  0001 C CNN
 F 3 "~" H 900 4750 50  0001 C CNN
 	1    900  4750
@@
 F 0 "R02" V 1693 4450 50  0000 C CNN
 F 1 "1k" V 1784 4450 50  0000 C CNN
-F 2 "" V 1830 4450 50  0001 C CNN
+F 2 "Resistor_THT:R_Axial_DIN0204_L3.6mm_D1.6mm_P5.08mm_Horizontal" V 1830 4450 50  0001 C CNN
 F 3 "~" H 1900 4450 50  0001 C CNN
 	1    1900 4450
@@
 F 0 "R01" H 1580 4604 50  0000 R CNN
 F 1 "2k" H 1580 4695 50  0000 R CNN
-F 2 "" V 1580 4650 50  0001 C CNN
+F 2 "Resistor_THT:R_Axial_DIN0204_L3.6mm_D1.6mm_P5.08mm_Horizontal" V 1580 4650 50  0001 C CNN
 F 3 "~" H 1650 4650 50  0001 C CNN
 	1    1650 4650
@@
 F 0 "R5" H 2020 2646 50  0000 L CNN
 F 1 "10k" H 2020 2555 50  0000 L CNN
-F 2 "" V 1880 2600 50  0001 C CNN
+F 2 "Resistor_THT:R_Axial_DIN0204_L3.6mm_D1.6mm_P5.08mm_Horizontal" V 1880 2600 50  0001 C CNN
 F 3 "~" H 1950 2600 50  0001 C CNN
 	1    1950 2600
@@
 F 0 "Rcal1" V 2343 1950 50  0000 C CNN
 F 1 "Rcal1" V 2434 1950 50  0000 C CNN
-F 2 "" V 2480 1950 50  0001 C CNN
+F 2 "Resistor_THT:R_Axial_DIN0204_L3.6mm_D1.6mm_P5.08mm_Horizontal" V 2480 1950 50  0001 C CNN
 F 3 "~" H 2550 1950 50  0001 C CNN
 	1    2550 1950
@@
 F 0 "Rcal2" V 1993 1950 50  0000 C CNN
 F 1 "Rcal2" V 2084 1950 50  0000 C CNN
-F 2 "" V 2130 1950 50  0001 C CNN
+F 2 "Resistor_THT:R_Axial_DIN0204_L3.6mm_D1.6mm_P5.08mm_Horizontal" V 2130 1950 50  0001 C CNN
 F 3 "~" H 2200 1950 50  0001 C CNN
 	1    2200 1950
@@
 $EndComp
 $Comp
-L Gaz-sensor:LTC1050 U1
+L iss_mosh_gaz_sensor-rescue:LTC1050-Gaz-sensor U1
 U 1 1 5BF8822B
 P 3200 2350
 F 0 "U1" H 3450 2250 50  0000 L CNN
 F 1 "LTC1050" H 3300 2150 50  0000 L CNN
-F 2 "" H 2750 2750 50  0001 C CNN
+F 2 "Package_DIP:DIP-8_W7.62mm_LongPads" H 2750 2750 50  0001 C CNN
 F 3 "" H 2750 2750 50  0001 C CNN
 	1    3200 2350
@@
 F 0 "R1" H 2670 2646 50  0000 L CNN
 F 1 "100k" H 2670 2555 50  0000 L CNN
-F 2 "" V 2530 2600 50  0001 C CNN
+F 2 "Resistor_THT:R_Axial_DIN0204_L3.6mm_D1.6mm_P5.08mm_Horizontal" V 2530 2600 50  0001 C CNN
 F 3 "~" H 2600 2600 50  0001 C CNN
 	1    2600 2600
@@
 F 0 "C1" H 2135 2554 50  0000 R CNN
 F 1 "100n" H 2135 2645 50  0000 R CNN
-F 2 "" H 2288 2450 50  0001 C CNN
+F 2 "Capacitor_THT:CP_Axial_L10.0mm_D4.5mm_P15.00mm_Horizontal" H 2288 2450 50  0001 C CNN
 F 3 "~" H 2250 2600 50  0001 C CNN
 	1    2250 2600
@@
 F 0 "C3" H 3465 1696 50  0000 L CNN
 F 1 "100n" H 3465 1605 50  0000 L CNN
-F 2 "" H 3388 1500 50  0001 C CNN
+F 2 "Capacitor_THT:CP_Axial_L10.0mm_D4.5mm_P15.00mm_Horizontal" H 3388 1500 50  0001 C CNN
 F 3 "~" H 3350 1650 50  0001 C CNN
 	1    3350 1650
@@
 F 0 "C4" H 4065 2246 50  0000 L CNN
 F 1 "1u" H 4065 2155 50  0000 L CNN
-F 2 "" H 3988 2050 50  0001 C CNN
+F 2 "Capacitor_THT:CP_Axial_L10.0mm_D4.5mm_P15.00mm_Horizontal" H 3988 2050 50  0001 C CNN
 F 3 "~" H 3950 2200 50  0001 C CNN
 	1    3950 2200
@@
 F 0 "R3" H 4370 2246 50  0000 L CNN
 F 1 "100k" H 4370 2155 50  0000 L CNN
-F 2 "" V 4230 2200 50  0001 C CNN
+F 2 "Resistor_THT:R_Axial_DIN0204_L3.6mm_D1.6mm_P5.08mm_Horizontal" V 4230 2200 50  0001 C CNN
 F 3 "~" H 4300 2200 50  0001 C CNN
 	1    4300 2200
@@
 F 0 "R6" V 4543 2050 50  0000 C CNN
 F 1 "1k" V 4634 2050 50  0000 C CNN
-F 2 "" V 4680 2050 50  0001 C CNN
+F 2 "Resistor_THT:R_Axial_DIN0204_L3.6mm_D1.6mm_P5.08mm_Horizontal" V 4680 2050 50  0001 C CNN
 F 3 "~" H 4750 2050 50  0001 C CNN
 	1    4750 2050
@@
 F 0 "C2" H 5115 2396 50  0000 L CNN
 F 1 "100n" H 5115 2305 50  0000 L CNN
-F 2 "" H 5038 2200 50  0001 C CNN
+F 2 "Capacitor_THT:CP_Axial_L10.0mm_D4.5mm_P15.00mm_Horizontal" H 5038 2200 50  0001 C CNN
 F 3 "~" H 5000 2350 50  0001 C CNN
 	1    5000 2350

Commit message: Capacitor
Parts:
- C1, C2, C3, C4: footprint Capacitor_THT:CP_Axial_L10.0mm_D4.5mm_P15.00mm_Horizontal -> Capacitor_THT:C_Disc_D3.0mm_W1.6mm_P2.50mm
Changed lines of the file:
@@
 F 0 "C1" H 2135 2554 50  0000 R CNN
 F 1 "100n" H 2135 2645 50  0000 R CNN
-F 2 "Capacitor_THT:CP_Axial_L10.0mm_D4.5mm_P15.00mm_Horizontal" H 2288 2450 50  0001 C CNN
+F 2 "Capacitor_THT:C_Disc_D3.0mm_W1.6mm_P2.50mm" H 2288 2450 50  0001 C CNN
 F 3 "~" H 2250 2600 50  0001 C CNN
 	1    2250 2600
@@
 F 0 "C3" H 3465 1696 50  0000 L CNN
 F 1 "100n" H 3465 1605 50  0000 L CNN
-F 2 "Capacitor_THT:CP_Axial_L10.0mm_D4.5mm_P15.00mm_Horizontal" H 3388 1500 50  0001 C CNN
+F 2 "Capacitor_THT:C_Disc_D3.0mm_W1.6mm_P2.50mm" H 3388 1500 50  0001 C CNN
 F 3 "~" H 3350 1650 50  0001 C CNN
 	1    3350 1650
@@
 F 0 "C4" H 4065 2246 50  0000 L CNN
 F 1 "1u" H 4065 2155 50  0000 L CNN
-F 2 "Capacitor_THT:CP_Axial_L10.0mm_D4.5mm_P15.00mm_Horizontal" H 3988 2050 50  0001 C CNN
+F 2 "Capacitor_THT:C_Disc_D3.0mm_W1.6mm_P2.50mm" H 3988 2050 50  0001 C CNN
 F 3 "~" H 3950 2200 50  0001 C CNN
 	1    3950 2200
@@
 F 0 "C2" H 5115 2396 50  0000 L CNN
 F 1 "100n" H 5115 2305 50  0000 L CNN
-F 2 "Capacitor_THT:CP_Axial_L10.0mm_D4.5mm_P15.00mm_Horizontal" H 5038 2200 50  0001 C CNN
+F 2 "Capacitor_THT:C_Disc_D3.0mm_W1.6mm_P2.50mm" H 5038 2200 50  0001 C CNN
 F 3 "~" H 5000 2350 50  0001 C CNN
 	1    5000 2350

Commit message: routage
Parts:
- added Rsensor1: 10k<...<1G, Socket_Arduino_Uno:TO-5-4(gas_sensor), symbol Device:R
Connections:
- net +3V3: now also Rsensor1.2
- net A0: no longer R5.2
- new net: R5.2, Rsensor1.1
Other:
- moved on the sheet: R5
Changed lines of the file:
@@
 Wire Wire Line
 	1500 1600 1200 1600
-Text Label 1950 3000 0    60   ~ 0
-A0
 Text Notes 1600 950  0    94   ~ 0
 Gaz Sensor
@@
 L Device:R R5
 U 1 1 5BF80849
-P 1950 2600
-F 0 "R5" H 2020 2646 50  0000 L CNN
-F 1 "10k" H 2020 2555 50  0000 L CNN
-F 2 "Resistor_THT:R_Axial_DIN0204_L3.6mm_D1.6mm_P5.08mm_Horizontal" V 1880 2600 50  0001 C CNN
-F 3 "~" H 1950 2600 50  0001 C CNN
-	1    1950 2600
-	1    0    0    -1
+P 1800 2450
+F 0 "R5" H 1870 2496 50  0000 L CNN
+F 1 "10k" H 1870 2405 50  0000 L CNN
+F 2 "Resistor_THT:R_Axial_DIN0204_L3.6mm_D1.6mm_P5.08mm_Horizontal" V 1730 2450 50  0001 C CNN
+F 3 "~" H 1800 2450 50  0001 C CNN
+	1    1800 2450
+	0    1    1    0
 $EndComp
 $Comp
@@
 Wire Wire Line
 	2600 2450 2250 2450
-Wire Wire Line
-	1950 2750 1950 3000
 $Comp
 L power:GND #PWR0111
@@
 	700  650  700  3200
 NoConn ~ 3250 2600
+$Comp
+L Device:R Rsensor1
+U 1 1 5C02A745
+P 1500 2450
+F 0 "Rsensor1" H 1570 2496 50  0000 L CNN
+F 1 "10k<...<1G" H 1570 2405 50  0000 L CNN
+F 2 "Socket_Arduino_Uno:TO-5-4(gas_sensor)" V 1430 2450 50  0001 C CNN
+F 3 "~" H 1500 2450 50  0001 C CNN
+	1    1500 2450
+	0    1    1    0
+$EndComp
+$Comp
+L power:+3.3V #PWR0113
+U 1 1 5C02CB80
+P 1300 2450
+F 0 "#PWR0113" H 1300 2300 50  0001 C CNN
+F 1 "+3.3V" V 1250 2500 50  0000 C CNN
+F 2 "" H 1300 2450 50  0000 C CNN
+F 3 "" H 1300 2450 50  0000 C CNN
+	1    1300 2450
+	0    -1   -1   0
+$EndComp
+Wire Wire Line
+	1350 2450 1300 2450
 $EndSCHEMATC
