File: iss_mosh_gaz_sensor.kicad_pcb (KiCad board)
At the start: 2 copper layers, 68.6 x 53.3 mm, 23 parts, among them J1 Conn_01x04, J2 Conn_01x08, P1 Power, P2 Analog, P3 Digital, P4 Digital, P5 CONN_01X01, P6 CONN_01X01, P7 CONN_01X01, P8 CONN_01X01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

Commit message: Capacitor
Parts:
- C1, C2, C3, C4: footprint Capacitor_THT:CP_Axial_L10.0mm_D4.5mm_P15.00mm_Horizontal -> Capacitor_THT:C_Disc_D3.0mm_W1.6mm_P2.50mm
- moved C3 24.8 mm to (151.0, 91.9)
- moved C1 20.4 mm to (146.4, 91.9)
- moved C2 5.77 mm to (146.4, 94.0)
- moved C4 4.51 mm to (151.0, 94.0)

Commit message: routage
Parts:
- added REF**: TO-5-4(gas_sensor), Socket_Arduino_Uno:TO-5-4(gas_sensor), F.Cu at (136.4, 116.2)
- moved R3 34.2 mm to (151.6, 93.3), turned to 90 degrees
- moved R6 32.0 mm to (151.6, 83.2), turned to 180 degrees
- moved Rcal2 22.9 mm to (133.9, 87.0), turned to 90 degrees
- moved R1 22.9 mm to (147.8, 106.0), turned to 90 degrees
- moved Rcal1 22.6 mm to (128.8, 89.5), turned to 90 degrees
- moved R01 17.3 mm to (165.6, 97.2), turned to 90 degrees
- moved C1 15.0 mm to (141.5, 106.0), turned to 270 degrees
- moved C2 13.5 mm to (147.8, 80.6), turned to 180 degrees
- moved R5 13.4 mm to (130.0, 103.5), turned to 270 degrees
- moved C3 12.5 mm to (140.2, 85.7), turned to 90 degrees
- moved R02 8.03 mm to (165.6, 83.2)
- moved J1 8.03 mm to (159.3, 111.1), turned to 0 degrees
- moved U1 7.73 mm to (133.9, 99.7), turned to 90 degrees
- moved C4 4.86 mm to (155.4, 92.0), turned to 90 degrees
Routing:
- net GND: track 0.00 -> 117.7 mm
- net +5V: track 11.2 -> 85.5 mm
- net +3V3: track 52.2 -> 0.00 mm
- net Net-(C4-Pad1): track 0.00 -> 35.8 mm
- net Net-(J2-Pad7): track 33.3 -> 3.81 mm
- net Net-(C1-Pad2): track 0.00 -> 29.1 mm
- net Net-(C4-Pad2): track 0.00 -> 23.6 mm
- net arduino: track 0.00 -> 14.9 mm
- net /A0: track 5.08 -> 14.7 mm
- net /6_UART_TX: track 17.6 -> 10.3 mm
- net Net-(Rcal1-Pad2): track 0.00 -> 6.13 mm
- net /7_UART_RX: track 52.5 -> 46.5 mm
Other:
- net class Default: clearance 0.2 -> 0.4; trace_width 0.25 -> 0.8; via_dia 0.6 -> 1.6; via_drill 0.4 -> 0.8
- rule trace_clearance: 0.2 -> 0.4
- rule trace_min: 0.2 -> 0.8

Commit message: Routage
Parts:
- removed REF**: TO-5-4(gas_sensor), Socket_Arduino_Uno:TO-5-4(gas_sensor)
- added Rsensor1: 10k<...<1G, Socket_Arduino_Uno:TO-5-4(gas_sensor), F.Cu at (131.3, 116.2)
- moved R01 5.08 mm to (170.7, 97.2)
Connections:
- R5 pad 2: /A0 -> Net-(R5-Pad2)
Routing:
- net Net-(J2-Pad7): track 3.81 -> 32.5 mm
- net +3V3: track 0.00 -> 16.9 mm
- net GND: track 117.7 -> 106.9 mm
- net Net-(R5-Pad2): track 0.00 -> 10.2 mm
- net +5V: track 85.5 -> 91.2 mm

Commit message: masse
Routing:
- added copper zone on B.Cu, net (none)
Changed lines of the file:
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@@
-(kicad_pcb (version 20171130) (host pcbnew "(5.0.1)-3")
+(kicad_pcb (version 20171130) (host pcbnew "(5.0.1)-4")
   (general
     (thickness 1.6)
@@
     (aux_axis_origin 110.998 126.365)
     (grid_origin 110.998 126.365)
-    (visible_elements 7FFFFFFF)
+    (visible_elements 7FFFF7FF)
     (pcbplotparams
       (layerselection 0x00030_80000001)
@@
   (segment (start 128.778 111.125) (end 130.048 109.855) (width 0.8) (layer F.Cu) (net 46))
   (segment (start 130.048 109.855) (end 130.048 108.585) (width 0.8) (layer F.Cu) (net 46))
+  (zone (net 0) (net_name "") (layer B.Cu) (hatch edge 0.508)
+    (connect_pads (clearance 0.508))
+    (min_thickness 0.254)
+    (fill yes (arc_segments 16) (thermal_gap 0.508) (thermal_bridge_width 0.508))
+    (polygon
+      (pts
+        (xy 109.728 71.755) (xy 109.728 127.635) (xy 180.848 127.635) (xy 180.848 71.755)
+      )
+    )
+  )
 )
